Commit message: fix(description): use separate xacro files for left and right hand models
- Add left.urdf.xacro and right.urdf.xacro as independent files
- Each hand uses its own correct joint parameters (origin xyz/rpy)
- Each hand uses its own mesh paths
- Update launch files to process new xacro files
- Remove old unified wujihand.urdf.xacro file

Resolve f-6599905232

File: wujihand_description/urdf/right.urdf.xacro (robot description, xacro)
@@ -1,10 +1,8 @@
 <?xml version="1.0" encoding="utf-8"?>
-<robot xmlns:xacro="http://www.ros.org/wiki/xacro" name="wujihand">
+<robot xmlns:xacro="http://www.ros.org/wiki/xacro" name="wujihand-right">
   <!-- Arguments -->
   <xacro:arg name="prefix" default="" />
-  <xacro:arg name="hand_type" default="right" />
   <!-- Properties -->
   <xacro:property name="prefix" value="$(arg prefix)" />
-  <xacro:property name="hand_type" value="$(arg hand_type)" />
   <!-- Material -->
   <material name="wujihand_gray">
@@ -22,12 +20,12 @@
       <origin xyz="0 0 0" rpy="0 0 0" />
       <geometry>
-        <mesh filename="package://wujihand_description/meshes/${hand_type}/palm_link.STL" />
-      </geometry>
-      <material name="wujihand_gray" />
-    </visual>
-    <collision>
-      <origin xyz="0 0 0" rpy="0 0 0" />
-      <geometry>
-        <mesh filename="package://wujihand_description/meshes/${hand_type}/palm_link_collision.STL" />
+        <mesh filename="package://wujihand_description/meshes/right/palm_link.STL" />
+      </geometry>
+      <material name="wujihand_gray" />
+    </visual>
+    <collision>
+      <origin xyz="0 0 0" rpy="0 0 0" />
+      <geometry>
+        <mesh filename="package://wujihand_description/meshes/right/palm_link.STL" />
       </geometry>
     </collision>
@@ -44,12 +42,12 @@
       <origin xyz="0 0 0" rpy="0 0 0" />
       <geometry>
-        <mesh filename="package://wujihand_description/meshes/${hand_type}/finger1_link1.STL" />
-      </geometry>
-      <material name="wujihand_gray" />
-    </visual>
-    <collision>
-      <origin xyz="0 0 0" rpy="0 0 0" />
-      <geometry>
-        <mesh filename="package://wujihand_description/meshes/${hand_type}/finger1_link1_collision.STL" />
+        <mesh filename="package://wujihand_description/meshes/right/finger1_link1.STL" />
+      </geometry>
+      <material name="wujihand_gray" />
+    </visual>
+    <collision>
+      <origin xyz="0 0 0" rpy="0 0 0" />
+      <geometry>
+        <mesh filename="package://wujihand_description/meshes/right/finger1_link1.STL" />
       </geometry>
     </collision>
@@ -72,12 +70,12 @@
       <origin xyz="0 0 0" rpy="0 0 0" />
       <geometry>
-        <mesh filename="package://wujihand_description/meshes/${hand_type}/finger1_link2.STL" />
-      </geometry>
-      <material name="wujihand_gray" />
-    </visual>
-    <collision>
-      <origin xyz="0 0 0" rpy="0 0 0" />
-      <geometry>
-        <mesh filename="package://wujihand_description/meshes/${hand_type}/finger1_link2_collision.STL" />
+        <mesh filename="package://wujihand_description/meshes/right/finger1_link2.STL" />
+      </geometry>
+      <material name="wujihand_gray" />
+    </visual>
+    <collision>
+      <origin xyz="0 0 0" rpy="0 0 0" />
+      <geometry>
+        <mesh filename="package://wujihand_description/meshes/right/finger1_link2.STL" />
       </geometry>
     </collision>
@@ -100,12 +98,12 @@
       <origin xyz="0 0 0" rpy="0 0 0" />
       <geometry>
-        <mesh filename="package://wujihand_description/meshes/${hand_type}/finger1_link3.STL" />
-      </geometry>
-      <material name="wujihand_gray" />
-    </visual>
-    <collision>
-      <origin xyz="0 0 0" rpy="0 0 0" />
-      <geometry>
-        <mesh filename="package://wujihand_description/meshes/${hand_type}/finger1_link3_collision.STL" />
+        <mesh filename="package://wujihand_description/meshes/right/finger1_link3.STL" />
+      </geometry>
+      <material name="wujihand_gray" />
+    </visual>
+    <collision>
+      <origin xyz="0 0 0" rpy="0 0 0" />
+      <geometry>
+        <mesh filename="package://wujihand_description/meshes/right/finger1_link3.STL" />
       </geometry>
     </collision>
@@ -128,12 +126,12 @@
       <origin xyz="0 0 0" rpy="0 0 0" />
       <geometry>
-        <mesh filename="package://wujihand_description/meshes/${hand_type}/finger1_link4.STL" />
-      </geometry>
-      <material name="wujihand_gray" />
-    </visual>
-    <collision>
-      <origin xyz="0 0 0" rpy="0 0 0" />
-      <geometry>
-        <mesh filename="package://wujihand_description/meshes/${hand_type}/finger1_link4_collision.STL" />
+        <mesh filename="package://wujihand_description/meshes/right/finger1_link4.STL" />
+      </geometry>
+      <material name="wujihand_gray" />
+    </visual>
+    <collision>
+      <origin xyz="0 0 0" rpy="0 0 0" />
+      <geometry>
+        <mesh filename="package://wujihand_description/meshes/right/finger1_link4.STL" />
       </geometry>
     </collision>
@@ -156,12 +154,12 @@
       <origin xyz="0 0 0" rpy="0 0 0" />
       <geometry>
-        <mesh filename="package://wujihand_description/meshes/${hand_type}/finger1_tip_link.STL" />
-      </geometry>
-      <material name="wujihand_gray" />
-    </visual>
-    <collision>
-      <origin xyz="0 0 0" rpy="0 0 0" />
-      <geometry>
-        <mesh filename="package://wujihand_description/meshes/${hand_type}/finger1_tip_link_collision.STL" />
+        <mesh filename="package://wujihand_description/meshes/right/finger1_tip_link.STL" />
+      </geometry>
+      <material name="wujihand_gray" />
+    </visual>
+    <collision>
+      <origin xyz="0 0 0" rpy="0 0 0" />
+      <geometry>
+        <mesh filename="package://wujihand_description/meshes/right/finger1_tip_link.STL" />
       </geometry>
     </collision>
@@ -183,12 +181,12 @@
       <origin xyz="0 0 0" rpy="0 0 0" />
       <geometry>
-        <mesh filename="package://wujihand_description/meshes/${hand_type}/finger2_link1.STL" />
-      </geometry>
-      <material name="wujihand_gray" />
-    </visual>
-    <collision>
-      <origin xyz="0 0 0" rpy="0 0 0" />
-      <geometry>
-        <mesh filename="package://wujihand_description/meshes/${hand_type}/finger2_link1_collision.STL" />
+        <mesh filename="package://wujihand_description/meshes/right/finger2_link1.STL" />
+      </geometry>
+      <material name="wujihand_gray" />
+    </visual>
+    <collision>
+      <origin xyz="0 0 0" rpy="0 0 0" />
+      <geometry>
+        <mesh filename="package://wujihand_description/meshes/right/finger2_link1.STL" />
       </geometry>
     </collision>
@@ -211,12 +209,12 @@
       <origin xyz="0 0 0" rpy="0 0 0" />
       <geometry>
-        <mesh filename="package://wujihand_description/meshes/${hand_type}/finger2_link2.STL" />
-      </geometry>
-      <material name="wujihand_gray" />
-    </visual>
-    <collision>
-      <origin xyz="0 0 0" rpy="0 0 0" />
-      <geometry>
-        <mesh filename="package://wujihand_description/meshes/${hand_type}/finger2_link2_collision.STL" />
+        <mesh filename="package://wujihand_description/meshes/right/finger2_link2.STL" />
+      </geometry>
+      <material name="wujihand_gray" />
+    </visual>
+    <collision>
+      <origin xyz="0 0 0" rpy="0 0 0" />
+      <geometry>
+        <mesh filename="package://wujihand_description/meshes/right/finger2_link2.STL" />
       </geometry>
     </collision>
@@ -239,12 +237,12 @@
       <origin xyz="0 0 0" rpy="0 0 0" />
       <geometry>
-        <mesh filename="package://wujihand_description/meshes/${hand_type}/finger2_link3.STL" />
-      </geometry>
-      <material name="wujihand_gray" />
-    </visual>
-    <collision>
-      <origin xyz="0 0 0" rpy="0 0 0" />
-      <geometry>
-        <mesh filename="package://wujihand_description/meshes/${hand_type}/finger2_link3_collision.STL" />
+        <mesh filename="package://wujihand_description/meshes/right/finger2_link3.STL" />
+      </geometry>
+      <material name="wujihand_gray" />
+    </visual>
+    <collision>
+      <origin xyz="0 0 0" rpy="0 0 0" />
+      <geometry>
+        <mesh filename="package://wujihand_description/meshes/right/finger2_link3.STL" />
       </geometry>
     </collision>
@@ -267,12 +265,12 @@
       <origin xyz="0 0 0" rpy="0 0 0" />
       <geometry>
-        <mesh filename="package://wujihand_description/meshes/${hand_type}/finger2_link4.STL" />
-      </geometry>
-      <material name="wujihand_gray" />
-    </visual>
-    <collision>
-      <origin xyz="0 0 0" rpy="0 0 0" />
-      <geometry>
-        <mesh filename="package://wujihand_description/meshes/${hand_type}/finger2_link4_collision.STL" />
+        <mesh filename="package://wujihand_description/meshes/right/finger2_link4.STL" />
+      </geometry>
+      <material name="wujihand_gray" />
+    </visual>
+    <collision>
+      <origin xyz="0 0 0" rpy="0 0 0" />
+      <geometry>
+        <mesh filename="package://wujihand_description/meshes/right/finger2_link4.STL" />
       </geometry>
     </collision>
@@ -295,12 +293,12 @@
       <origin xyz="0 0 0" rpy="0 0 0" />
       <geometry>
-        <mesh filename="package://wujihand_description/meshes/${hand_type}/finger2_tip_link.STL" />
-      </geometry>
-      <material name="wujihand_gray" />
-    </visual>
-    <collision>
-      <origin xyz="0 0 0" rpy="0 0 0" />
-      <geometry>
-        <mesh filename="package://wujihand_description/meshes/${hand_type}/finger2_tip_link_collision.STL" />
+        <mesh filename="package://wujihand_description/meshes/right/finger2_tip_link.STL" />
+      </geometry>
+      <material name="wujihand_gray" />
+    </visual>
+    <collision>
+      <origin xyz="0 0 0" rpy="0 0 0" />
+      <geometry>
+        <mesh filename="package://wujihand_description/meshes/right/finger2_tip_link.STL" />
       </geometry>
     </collision>
@@ -322,12 +320,12 @@
       <origin xyz="0 0 0" rpy="0 0 0" />
       <geometry>
-        <mesh filename="package://wujihand_description/meshes/${hand_type}/finger3_link1.STL" />
-      </geometry>
-      <material name="wujihand_gray" />
-    </visual>
-    <collision>
-      <origin xyz="0 0 0" rpy="0 0 0" />
-      <geometry>
-        <mesh filename="package://wujihand_description/meshes/${hand_type}/finger3_link1_collision.STL" />
+        <mesh filename="package://wujihand_description/meshes/right/finger3_link1.STL" />
+      </geometry>
+      <material name="wujihand_gray" />
+    </visual>
+    <collision>
+      <origin xyz="0 0 0" rpy="0 0 0" />
+      <geometry>
+        <mesh filename="package://wujihand_description/meshes/right/finger3_link1.STL" />
       </geometry>
     </collision>
@@ -350,12 +348,12 @@
       <origin xyz="0 0 0" rpy="0 0 0" />
       <geometry>
-        <mesh filename="package://wujihand_description/meshes/${hand_type}/finger3_link2.STL" />
-      </geometry>
-      <material name="wujihand_gray" />
-    </visual>
-    <collision>
-      <origin xyz="0 0 0" rpy="0 0 0" />
-      <geometry>
-        <mesh filename="package://wujihand_description/meshes/${hand_type}/finger3_link2_collision.STL" />
+        <mesh filename="package://wujihand_description/meshes/right/finger3_link2.STL" />
+      </geometry>
+      <material name="wujihand_gray" />
+    </visual>
+    <collision>
+      <origin xyz="0 0 0" rpy="0 0 0" />
+      <geometry>
+        <mesh filename="package://wujihand_description/meshes/right/finger3_link2.STL" />
       </geometry>
     </collision>
@@ -378,12 +376,12 @@
       <origin xyz="0 0 0" rpy="0 0 0" />
       <geometry>
-        <mesh filename="package://wujihand_description/meshes/${hand_type}/finger3_link3.STL" />
-      </geometry>
-      <material name="wujihand_gray" />
-    </visual>
-    <collision>
-      <origin xyz="0 0 0" rpy="0 0 0" />
-      <geometry>
-        <mesh filename="package://wujihand_description/meshes/${hand_type}/finger3_link3_collision.STL" />
+        <mesh filename="package://wujihand_description/meshes/right/finger3_link3.STL" />
+      </geometry>
+      <material name="wujihand_gray" />
+    </visual>
+    <collision>
+      <origin xyz="0 0 0" rpy="0 0 0" />
+      <geometry>
+        <mesh filename="package://wujihand_description/meshes/right/finger3_link3.STL" />
       </geometry>
     </collision>
@@ -406,12 +404,12 @@
       <origin xyz="0 0 0" rpy="0 0 0" />
       <geometry>
-        <mesh filename="package://wujihand_description/meshes/${hand_type}/finger3_link4.STL" />
-      </geometry>
-      <material name="wujihand_gray" />
-    </visual>
-    <collision>
-      <origin xyz="0 0 0" rpy="0 0 0" />
-      <geometry>
-        <mesh filename="package://wujihand_description/meshes/${hand_type}/finger3_link4_collision.STL" />
+        <mesh filename="package://wujihand_description/meshes/right/finger3_link4.STL" />
+      </geometry>
+      <material name="wujihand_gray" />
+    </visual>
+    <collision>
+      <origin xyz="0 0 0" rpy="0 0 0" />
+      <geometry>
+        <mesh filename="package://wujihand_description/meshes/right/finger3_link4.STL" />
       </geometry>
     </collision>
@@ -434,12 +432,12 @@
       <origin xyz="0 0 0" rpy="0 0 0" />
       <geometry>
-        <mesh filename="package://wujihand_description/meshes/${hand_type}/finger3_tip_link.STL" />
-      </geometry>
-      <material name="wujihand_gray" />
-    </visual>
-    <collision>
-      <origin xyz="0 0 0" rpy="0 0 0" />
-      <geometry>
-        <mesh filename="package://wujihand_description/meshes/${hand_type}/finger3_tip_link_collision.STL" />
+        <mesh filename="package://wujihand_description/meshes/right/finger3_tip_link.STL" />
+      </geometry>
+      <material name="wujihand_gray" />
+    </visual>
+    <collision>
+      <origin xyz="0 0 0" rpy="0 0 0" />
+      <geometry>
+        <mesh filename="package://wujihand_description/meshes/right/finger3_tip_link.STL" />
       </geometry>
     </collision>
@@ -461,12 +459,12 @@
       <origin xyz="0 0 0" rpy="0 0 0" />
       <geometry>
-        <mesh filename="package://wujihand_description/meshes/${hand_type}/finger4_link1.STL" />
-      </geometry>
-      <material name="wujihand_gray" />
-    </visual>
-    <collision>
-      <origin xyz="0 0 0" rpy="0 0 0" />
-      <geometry>
-        <mesh filename="package://wujihand_description/meshes/${hand_type}/finger4_link1_collision.STL" />
+        <mesh filename="package://wujihand_description/meshes/right/finger4_link1.STL" />
+      </geometry>
+      <material name="wujihand_gray" />
+    </visual>
+    <collision>
+      <origin xyz="0 0 0" rpy="0 0 0" />
+      <geometry>
+        <mesh filename="package://wujihand_description/meshes/right/finger4_link1.STL" />
       </geometry>
     </collision>
@@ -489,12 +487,12 @@
       <origin xyz="0 0 0" rpy="0 0 0" />
       <geometry>
-        <mesh filename="package://wujihand_description/meshes/${hand_type}/finger4_link2.STL" />
-      </geometry>
-      <material name="wujihand_gray" />
-    </visual>
-    <collision>
-      <origin xyz="0 0 0" rpy="0 0 0" />
-      <geometry>
-        <mesh filename="package://wujihand_description/meshes/${hand_type}/finger4_link2_collision.STL" />
+        <mesh filename="package://wujihand_description/meshes/right/finger4_link2.STL" />
+      </geometry>
+      <material name="wujihand_gray" />
+    </visual>
+    <collision>
+      <origin xyz="0 0 0" rpy="0 0 0" />
+      <geometry>
+        <mesh filename="package://wujihand_description/meshes/right/finger4_link2.STL" />
       </geometry>
     </collision>
@@ -517,12 +515,12 @@
       <origin xyz="0 0 0" rpy="0 0 0" />
       <geometry>
-        <mesh filename="package://wujihand_description/meshes/${hand_type}/finger4_link3.STL" />
-      </geometry>
-      <material name="wujihand_gray" />
-    </visual>
-    <collision>
-      <origin xyz="0 0 0" rpy="0 0 0" />
-      <geometry>
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